Commit message: Modified the robot model (WIP)

File: urdf/ball.xacro (robot description, xacro)
@@ -1,5 +1,5 @@
 <?xml version="1.0"?>
 <robot xmlns:xacro="http://www.ros.org/wiki/xacro" name="ball">
-<xacro:include filename="$(find exp_assignment2)/urdf/ball.gazebo"/>
+<xacro:include filename="$(find erl_second_assignment)/urdf/ball.gazebo"/>
   <material name="black">
     <color rgba="0.0 0.0 0.0 1.0"/>

File: urdf/robot.xacro (robot description, xacro)
@@ -1,5 +1,5 @@
 <?xml version="1.0"?>
 <robot xmlns:xacro="http://www.ros.org/wiki/xacro" name="robot_xacro">
-<xacro:include filename="$(find exp_assignment2)/urdf/robot.gazebo"/>
+<xacro:include filename="$(find erl_second_assignment)/urdf/robot.gazebo"/>
 	<xacro:property name="length_wheel" value="0.04" />
 	<xacro:property name="radius_wheel" value="0.1" />
@@ -40,4 +40,5 @@
     <color rgba="1.0 1.0 1.0 1.0"/>
   </material>
+  <!-- Links -->
 	  <link name="link_chassis">
     <!-- pose and inertial -->
@@ -99,4 +100,67 @@
     </visual>
   </link>
+  <link name="link_neck">
+  	<inertial>
+  		<mass value="0.025"/>
+  		<origin xyz="0 0 0" rpy="0 0 0" />
+  		<inertia ixx="0.000010279" ixy="0" ixz="0" iyy="0.000010279" iyz="0" izz="0.000007225"/>
+  	</inertial>
+  	<collision>
+  	  <origin xyz="0 0 0.125" rpy="0 0 0"/>
+      <geometry>
+        <cylinder radius="0.06" length="0.25"/>
+      </geometry>
+  	</collision>
+  	<visual>
+  	  <origin xyz="0 0 0.125" rpy="0 0 0"/>
+      <geometry>
+        <cylinder radius="0.06" length="0.25"/>
+      </geometry>
+      <material name="red" />
+  	</visual>
+  </link>
+  <link name="link_head">
+  	<inertial>
+  		<mass value="0.1"/>
+  		<origin xyz="0 0 0" rpy="0 0 0" />
+  		<inertia ixx="0.0000416666667" ixy="0" ixz="0" iyy="0.0000416666667" iyz="0" izz="0.0000416666667"/>
+  	</inertial>
+  	<collision>
+  	  <origin xyz="0.025 0 0.05" rpy="0 0 0"/>
+      <geometry>
+        <box size="0.15 0.1 0.1"/>
+      </geometry>
+  	</collision>
+  	<visual>
+  	  <origin xyz="0.025 0 0.05" rpy="0 0 0"/>
+      <geometry>
+        <box size="0.15 0.1 0.1"/>
+      </geometry>
+      <material name="red" />
+  	</visual>
+  </link>
+  <link name="camera_link">
+	    <collision>
+	      <origin xyz="0 0 0.025" rpy="0 0 0"/>
+	      <geometry>
+		      <box size="0.05 0.05 0.05"/>
+	      </geometry>
+	    </collision>
+	    <visual>
+	      <origin xyz="0 0 0.025" rpy="0 0 0"/>
+	      <geometry>
+		      <box size="0.05 0.05 0.05"/>
+	      </geometry>
+	      <material name="red">
+		      <color rgba="1 0 0 1"/>
+	      </material>
+	    </visual>
+	    <inertial>
+	      <mass value="1e-5" />
+	      <origin xyz="0 0 0" rpy="0 0 0"/>
+	      <inertia ixx="1e-6" ixy="0" ixz="0" iyy="1e-6" iyz="0" izz="1e-6" />
+	    </inertial>
+  </link>
+  <!-- Joints -->
   <joint name="joint_right_wheel" type="continuous">
     <origin rpy="0 0 0" xyz="-0.05 0.15 0"/>
@@ -115,30 +179,22 @@
     <joint_properties damping="1.0" friction="1.0"/>
   </joint>
-  <link name="camera_link">
-	    <collision>
-	      <origin xyz="0 0 0.025" rpy="0 0 0"/>
-	      <geometry>
-		<box size="0.05 0.05 0.05"/>
-	      </geometry>
-	    </collision>
-	    <visual>
-	      <origin xyz="0 0 0.025" rpy="0 0 0"/>
-	      <geometry>
-		<box size="0.05 0.05 0.05"/>
-	      </geometry>
-	      <material name="red">
-		<color rgba="1 0 0 1"/>
-	      </material>
-	    </visual>
-	    <inertial>
-	      <mass value="1e-5" />
-	      <origin xyz="0 0 0" rpy="0 0 0"/>
-	      <inertia ixx="1e-6" ixy="0" ixz="0" iyy="1e-6" iyz="0" izz="1e-6" />
-	    </inertial>
-  </link>
+  <joint name="joint_neck" type="fixed">
+	    <axis xyz="0 1 0" />
+	    <origin xyz="0.15 0 0.05" rpy="0 0 0"/>
+	    <parent link="link_chassis"/>
+	    <child link="link_neck"/>
+	 </joint>
+  <joint name="joint_head" type="continuous">
+    <origin rpy="0 0 0" xyz="0 0 0.125"/>
+    <child link="link_head"/>
+    <parent link="link_neck"/>
+    <axis rpy="0 0 0" xyz="0 0 1"/>
+    <limit effort="10000" velocity="1000"/>
+    <joint_properties damping="1.0" friction="1.0"/>
+  </joint>
   <joint name="camera_joint" type="fixed">
 	    <axis xyz="0 1 0" />
-	    <origin xyz="0.23 0 0.0" rpy="0 0 0"/>
-	    <parent link="link_chassis"/>
+	    <origin xyz="0.047 0 0.025" rpy="0 0 0"/>
+	    <parent link="link_head"/>
 	    <child link="camera_link"/>
 	 </joint>
