Commit message: Robot model and action server, person module and changes in the files
Completed the robot model, added the robot's action server, added the person module, modified the launchfile and the CMakeLists

File: urdf/robot.xacro (robot description, xacro)
@@ -127,5 +127,5 @@
   	</inertial>
   	<collision>
-  	  <origin xyz="0.025 0 0.05" rpy="0 0 0"/>
+  	  <origin xyz="0.05 0 0.05" rpy="0 0 0"/>
       <geometry>
         <box size="0.15 0.1 0.1"/>
@@ -133,5 +133,5 @@
   	</collision>
   	<visual>
-  	  <origin xyz="0.025 0 0.05" rpy="0 0 0"/>
+  	  <origin xyz="0.05 0 0.05" rpy="0 0 0"/>
       <geometry>
         <box size="0.15 0.1 0.1"/>
@@ -181,10 +181,10 @@
   <joint name="joint_neck" type="fixed">
 	    <axis xyz="0 1 0" />
-	    <origin xyz="0.15 0 0.05" rpy="0 0 0"/>
+	    <origin xyz="0.15 0 0.035" rpy="0 0 0"/>
 	    <parent link="link_chassis"/>
 	    <child link="link_neck"/>
 	 </joint>
   <joint name="joint_head" type="continuous">
-    <origin rpy="0 0 0" xyz="0 0 0.125"/>
+    <origin rpy="0 0 0" xyz="0 0 0.25"/>
     <child link="link_head"/>
     <parent link="link_neck"/>
@@ -195,5 +195,5 @@
   <joint name="camera_joint" type="fixed">
 	    <axis xyz="0 1 0" />
-	    <origin xyz="0.047 0 0.025" rpy="0 0 0"/>
+	    <origin xyz="0.11 0 0.06" rpy="0 0 0"/>
 	    <parent link="link_head"/>
 	    <child link="camera_link"/>

Commit message: Modified the programs and added the joint controller

File: urdf/robot.xacro (robot description, xacro)
@@ -199,3 +199,14 @@
 	    <child link="camera_link"/>
 	 </joint>
+  <!-- Transmissions -->
+  <transmission name="joint_head_trans">
+	  <type>transmission_interface/SimpleTransmission</type>
+	  <joint name="joint_head">
+		  <hardwareInterface>hardware_interface/EffortJointInterface</hardwareInterface>
+	  </joint>
+	  <actuator name="motor1">
+		  <hardwareInterface>hardware_interface/EffortJointInterface</hardwareInterface>
+		  <mechanicalInterface>1</mechanicalInterface>
+	  </actuator>
+  </transmission>
 </robot>

Commit message: Tested some behaviours and fixed some bugs

File: urdf/robot.xacro (robot description, xacro)
@@ -41,5 +41,5 @@
   </material>
   <!-- Links -->
-	  <link name="link_chassis">
+	<link name="link_chassis">
     <!-- pose and inertial -->
     <pose>0 0 0.1 0 0 0</pose>
@@ -76,5 +76,5 @@
     </visual>
   </link>
-   <link name="link_right_wheel">
+  <link name="link_right_wheel">
     <xacro:default_inertial mass="0.2"/>
     <collision name="link_right_wheel_collision">
@@ -88,5 +88,5 @@
     </visual>
   </link>
-   <link name="link_left_wheel">
+  <link name="link_left_wheel">
     <xacro:default_inertial mass="0.2"/>
     <collision name="link_left_wheel_collision">
@@ -117,5 +117,5 @@
         <cylinder radius="0.06" length="0.25"/>
       </geometry>
-      <material name="red" />
+      <material name="orange" />
   	</visual>
   </link>
@@ -137,5 +137,5 @@
         <box size="0.15 0.1 0.1"/>
       </geometry>
-      <material name="red" />
+      <material name="orange" />
   	</visual>
   </link>
@@ -180,9 +180,8 @@
   </joint>
   <joint name="joint_neck" type="fixed">
-	    <axis xyz="0 1 0" />
-	    <origin xyz="0.15 0 0.035" rpy="0 0 0"/>
-	    <parent link="link_chassis"/>
-	    <child link="link_neck"/>
-	 </joint>
+	  <origin xyz="0.15 0 0.035" rpy="0 0 0"/>
+	  <parent link="link_chassis"/>
+	  <child link="link_neck"/>
+	</joint>
   <joint name="joint_head" type="continuous">
     <origin rpy="0 0 0" xyz="0 0 0.25"/>
@@ -194,9 +193,8 @@
   </joint>
   <joint name="camera_joint" type="fixed">
-	    <axis xyz="0 1 0" />
-	    <origin xyz="0.11 0 0.06" rpy="0 0 0"/>
-	    <parent link="link_head"/>
-	    <child link="camera_link"/>
-	 </joint>
+	  <origin xyz="0.11 0 0.06" rpy="0 0 0"/>
+	  <parent link="link_head"/>
+	  <child link="camera_link"/>
+	</joint>
   <!-- Transmissions -->
   <transmission name="joint_head_trans">

Commit message: Completed the assignment and carried out extensive testing

File: urdf/robot.xacro (robot description, xacro)
@@ -184,11 +184,10 @@
 	  <child link="link_neck"/>
 	</joint>
-  <joint name="joint_head" type="continuous">
-    <origin rpy="0 0 0" xyz="0 0 0.25"/>
-    <child link="link_head"/>
-    <parent link="link_neck"/>
-    <axis rpy="0 0 0" xyz="0 0 1"/>
-    <limit effort="10000" velocity="1000"/>
-    <joint_properties damping="1.0" friction="1.0"/>
+  <joint name="joint_head" type="revolute">
+    <axis xyz="0 0 1"/>
+  	<limit effort="1000.0" lower="-6.28" upper="6.28" velocity="0.2"/>
+  	<origin rpy="0 0 0" xyz="0 0 0.25"/>
+  	<parent link="link_neck"/>
+  	<child link="link_head"/>
   </joint>
   <joint name="camera_joint" type="fixed">
